Commit message: kinemetic_server

File: lab2/dummy_description/robot/dummy.xacro (robot description, xacro)
@@ -71,5 +71,5 @@
     <parent link="link_2"/>
     <child link="end_effector"/>
-    <origin rpy="1.57 0 1.57" xyz="0.16 0 0"/>
+    <origin rpy="-1.57 0 0" xyz="0.16 0 0"/>
     <axis xyz="0 0 1"/>
     <limit lower="-3.14" upper="3.14" effort="0.5" velocity="0.5"/>
